File: lpc1769_stick2board/lpc1769_stick2board.sch (KiCad schematic (older format))
At the start: 6 parts, among them J1 Conn_01x27, J2 Conn_01x27, J3 Conn_02x10_Odd_Even, U1 LPCXpresso_LPC1769_revB

Commit message: PLACA TERMINADA. LISTA PARA PLANCHAR
Parts:
- removed BT1: Battery_Cell, Battery_Holders:Keystone_106_1x20mm-CoinCell, symbol Battery_Cell
Changed lines of the file:
@@
-$EndComp
-$Comp
-L GND #PWR01
-U 1 1 5BC5F4F8
-P 2850 2350
-F 0 "#PWR01" H 2850 2100 50  0001 C CNN
-F 1 "GND" H 2850 2200 50  0000 C CNN
-F 2 "" H 2850 2350 50  0001 C CNN
-F 3 "" H 2850 2350 50  0001 C CNN
-	1    2850 2350
-	1    0    0    -1
 $EndComp
 $Comp
@@
 Text Label 4750 5900 1    60   ~ 0
 P14
-$Comp
-L Battery_Cell BT1
-U 1 1 5BC60F7F
-P 2850 2000
-F 0 "BT1" H 2950 2100 50  0000 L CNN
-F 1 "Battery_Cell" H 2950 2000 50  0000 L CNN
-F 2 "Battery_Holders:Keystone_106_1x20mm-CoinCell" V 2850 2060 50  0001 C CNN
-F 3 "" V 2850 2060 50  0001 C CNN
-	1    2850 2000
-	1    0    0    -1
-$EndComp
-$Comp
-L PWR_FLAG #FLG03
-U 1 1 5BC612D7
-P 2500 2150
-F 0 "#FLG03" H 2500 2225 50  0001 C CNN
-F 1 "PWR_FLAG" H 2500 2300 50  0000 C CNN
-F 2 "" H 2500 2150 50  0001 C CNN
-F 3 "" H 2500 2150 50  0001 C CNN
-	1    2500 2150
-	1    0    0    -1
-$EndComp
 Text Notes 4100 1350 0    60   ~ 12
 Módulo para conexión de LPCXpresso LPC1769 rev C
@@
 	7000 2350 7050 2350
 Wire Wire Line
-	2850 2100 2850 2350
-Wire Wire Line
-	2500 2200 3550 2200
-Wire Wire Line
-	3550 2200 3550 2350
-Connection ~ 3550 2350
-Wire Wire Line
 	6700 5050 6700 4950
 Connection ~ 6700 4950
@@
 Wire Wire Line
 	4250 5550 4250 5900
-Connection ~ 2850 2200
-Wire Wire Line
-	2850 1800 2850 1700
-Wire Wire Line
-	3750 1700 3750 2550
-Connection ~ 3750 2550
-Wire Wire Line
-	2500 2150 2500 2200
-Wire Wire Line
-	2850 1700 3750 1700
 Wire Wire Line
 	8850 2350 9150 2350
@@
 Text Notes 6350 1950 0    60   ~ 0
 Solo puentear en caso\nde no alimentar vía USB.
+$Comp
+L GND #PWR?
+U 1 1 5BC9F8CA
+P 2850 2350
+F 0 "#PWR?" H 2850 2100 50  0001 C CNN
+F 1 "GND" H 2850 2200 50  0000 C CNN
+F 2 "" H 2850 2350 50  0001 C CNN
+F 3 "" H 2850 2350 50  0001 C CNN
+	1    2850 2350
+	1    0    0    -1
+$EndComp
+Wire Wire Line
+	2850 2000 2850 2350
+Wire Wire Line
+	2850 2150 3650 2150
+Wire Wire Line
+	3650 2150 3650 2350
+Connection ~ 3650 2350
+$Comp
+L PWR_FLAG #FLG?
+U 1 1 5BC9F967
+P 2850 2000
+F 0 "#FLG?" H 2850 2075 50  0001 C CNN
+F 1 "PWR_FLAG" H 2850 2150 50  0000 C CNN
+F 2 "" H 2850 2000 50  0001 C CNN
+F 3 "" H 2850 2000 50  0001 C CNN
+	1    2850 2000
+	1    0    0    -1
+$EndComp
+Connection ~ 2850 2150
 $EndSCHEMATC
